File: hardware_design/ESP32-S3_6_Motor_Driver_IMU/ESP32-S3_6_Motor_Driver_IMU.kicad_sch (KiCad schematic)
At the start: 87 parts, among them J1 USB_C_Receptacle_USB2.0_16P, J2 Conn_01x10, J3 Conn_01x10, J4 Conn_01x01, SW1 3-1437565-0, SW2 3-1437565-0, U1 ESP32-S3-MINI-1, U2 LD39200PU33R, U3 LMR38020FDDAR, U4 TPS2116DRLR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

Commit message: Add diagram showing ROS2 usage
Also make fixes to schematic
Parts:
- J2: value Conn_01x10 -> Conn_01x09; footprint Connector_PinHeader_2.54mm:PinHeader_1x10_P2.54mm_Vertical -> Connector_PinHeader_2.54mm:PinHeader_1x09_P2.54mm_Vertical; symbol Connector_Generic:Conn_01x10 -> Connector_Generic:Conn_01x09
- J3: value Conn_01x10 -> Conn_01x09; symbol Connector_Generic:Conn_01x10 -> Connector_Generic:Conn_01x09
Connections:
- net 16: now also J3.1 (Pin_1); no longer J2.10 (Pin_10)
- net 39: now also J3.4 (Pin_4); no longer J3.5 (Pin_5)
- net 40: now also J3.5 (Pin_5); no longer J3.6 (Pin_6)
- net 41: now also J3.6 (Pin_6); no longer J3.7 (Pin_7)
- net 42: now also J3.7 (Pin_7); no longer J3.8 (Pin_8)
- net IMU_INT: now also U1.22 (IO18)
- net LOG/46: now also J3.9 (Pin_9); no longer J3.10 (Pin_10)
- net RST: no longer U6.11 (NRST)
- net RX/44: now also J3.3 (Pin_3); no longer J3.4 (Pin_4)
- net TX/43: now also J3.2 (Pin_2); no longer J3.3 (Pin_3)
- net VDD_SPI/45: now also J3.8 (Pin_8); no longer J3.9 (Pin_9)
- net 17 renamed IMU_RST
- net IMU_RST: now also U6.11 (NRST); no longer J3.1 (Pin_1)
- removed net 18: J3.2 (Pin_2), U1.22 (IO18)
Changed lines of the file:
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@@
 		)
 	)
+	(label "TX{slash}43"
+		(at 331.47 25.4 180)
+		(effects
+			(font
+				(size 1.27 1.27)
+			)
+			(justify right bottom)
+		)
+	)
 	(label "OUT2"
 		(at 186.69 129.54 0)
@@
 		)
 	)
-	(label "RX{slash}44"
-		(at 331.47 30.48 180)
-		(effects
-			(font
-				(size 1.27 1.27)
-			)
-			(justify right bottom)
-		)
-	)
 	(label "PICO{slash}11"
 		(at 238.76 78.74 180)
@@
 		)
 	)
-	(label "41"
-		(at 331.47 38.1 180)
+	(label "40"
+		(at 331.47 33.02 180)
 		(effects
 			(font
@@
 		)
 	)
-	(label "40"
-		(at 331.47 35.56 180)
-		(effects
-			(font
-				(size 1.27 1.27)
-			)
-			(justify right bottom)
-		)
-	)
 	(label "D-"
 		(at 45.72 45.72 0)
@@
 		)
 	)
-	(label "42"
-		(at 331.47 40.64 180)
-		(effects
-			(font
-				(size 1.27 1.27)
-			)
-			(justify right bottom)
-		)
-	)
 	(label "33"
 		(at 326.39 119.38 180)
@@
 		)
 	)
-	(label "18"
-		(at 331.47 25.4 180)
-		(effects
-			(font
-				(size 1.27 1.27)
-			)
-			(justify right bottom)
-		)
-	)
 	(label "IMU_INT"
 		(at 135.89 66.04 180)
@@
 		)
 	)
-	(label "17"
-		(at 331.47 22.86 180)
+	(label "RX{slash}44"
+		(at 331.47 27.94 180)
 		(effects
 			(font
@@
 		)
 	)
+	(label "41"
+		(at 331.47 35.56 180)
+		(effects
+			(font
+				(size 1.27 1.27)
+			)
+			(justify right bottom)
+		)
+	)
 	(label "PICO{slash}11"
 		(at 151.13 137.16 180)
@@
 		)
 	)
-	(label "TX{slash}43"
-		(at 331.47 27.94 180)
+	(label "IMU_RST"
+		(at 135.89 58.42 180)
 		(effects
 			(font
@@
 		)
 	)
-	(label "RST"
-		(at 135.89 58.42 180)
+	(label "47"
+		(at 151.13 154.94 180)
 		(effects
 			(font
@@
 		)
 	)
-	(label "47"
-		(at 151.13 154.94 180)
+	(label "OUT8"
+		(at 337.82 104.14 180)
 		(effects
 			(font
@@
 		)
 	)
-	(label "OUT8"
-		(at 337.82 104.14 180)
+	(label "39"
+		(at 331.47 30.48 180)
 		(effects
 			(font
@@
 		)
 	)
-	(label "40"
-		(at 269.24 81.28 0)
+	(label "VDD_SPI{slash}45"
+		(at 331.47 40.64 180)
 		(effects
 			(font
 				(size 1.27 1.27)
 			)
-			(justify left bottom)
+			(justify right bottom)
 		)
 	)
-	(label "39"
-		(at 331.47 33.02 180)
+	(label "40"
+		(at 269.24 81.28 0)
 		(effects
 			(font
 				(size 1.27 1.27)
 			)
-			(justify right bottom)
+			(justify left bottom)
 		)
 	)
@@
 		)
 	)
-	(label "16"
-		(at 304.8 45.72 180)
-		(effects
-			(font
-				(size 1.27 1.27)
-			)
-			(justify right bottom)
-		)
-	)
 	(label "35"
 		(at 269.24 68.58 0)
@@
 		)
 	)
+	(label "42"
+		(at 331.47 38.1 180)
+		(effects
+			(font
+				(size 1.27 1.27)
+			)
+			(justify right bottom)
+		)
+	)
 	(label "D+"
 		(at 269.24 55.88 0)
@@
 		)
 	)
-	(label "17"
+	(label "IMU_RST"
 		(at 238.76 93.98 180)
 		(effects
@@
 		)
 	)
-	(label "LOG{slash}46"
-		(at 331.47 45.72 180)
-		(effects
-			(font
-				(size 1.27 1.27)
-			)
-			(justify right bottom)
-		)
-	)
 	(label "48"
 		(at 269.24 96.52 0)
@@
 		)
 	)
-	(label "VDD_SPI{slash}45"
-		(at 331.47 43.18 180)
-		(effects
-			(font
-				(size 1.27 1.27)
-			)
-			(justify right bottom)
-		)
-	)
 	(label "OUT9"
 		(at 306.07 138.43 180)
@@
 		)
 	)
-	(label "18"
+	(label "IMU_INT"
 		(at 238.76 96.52 180)
 		(effects
@@
 		)
 	)
+	(label "LOG{slash}46"
+		(at 331.47 43.18 180)
+		(effects
+			(font
+				(size 1.27 1.27)
+			)
+			(justify right bottom)
+		)
+	)
 	(label "OUT4"
 		(at 151.13 152.4 180)
@@
 		)
 	)
+	(label "16"
+		(at 331.47 22.86 180)
+		(effects
+			(font
+				(size 1.27 1.27)
+			)
+			(justify right bottom)
+		)
+	)
 	(label "48"
 		(at 151.13 144.78 180)
@@
 	)
 	(symbol
-		(lib_id "Connector_Generic:Conn_01x10")
+		(lib_id "Connector_Generic:Conn_01x09")
 		(at 309.88 33.02 0)
 		(unit 1)
@@
 		(fields_autoplaced yes)
 		(property "Reference" "J2"
-			(at 312.42 33.0199 0)
+			(at 312.42 31.7499 0)
 			(effects
 				(font
@@
 			)
 		)
-		(property "Value" "Conn_01x10"
-			(at 312.42 35.5599 0)
+		(property "Value" "Conn_01x09"
+			(at 312.42 34.2899 0)
 			(effects
 				(font
@@
 			)
 		)
-		(property "Footprint" "Connector_PinHeader_2.54mm:PinHeader_1x10_P2.54mm_Vertical"
+		(property "Footprint" "Connector_PinHeader_2.54mm:PinHeader_1x09_P2.54mm_Vertical"
 			(at 309.88 33.02 0)
 			(effects
@@
 			)
 		)
-		(property "Description" "Generic connector, single row, 01x10, script generated (kicad-library-utils/schlib/autogen/connector/)"
+		(property "Description" "Generic connector, single row, 01x09, script generated (kicad-library-utils/schlib/autogen/connector/)"
 			(at 309.88 33.02 0)
 			(effects
@@
 		(pin "2"
 		)
-		(pin "10"
-		)
 		(instances
 			(project ""
@@
 	)
 	(symbol
-		(lib_id "Connector_Generic:Conn_01x10")
+		(lib_id "Connector_Generic:Conn_01x09")
 		(at 336.55 33.02 0)
 		(unit 1)
@@
 		(fields_autoplaced yes)
 		(property "Reference" "J3"
-			(at 339.09 33.0199 0)
+			(at 339.09 31.7499 0)
 			(effects
 				(font
@@
 			)
 		)
-		(property "Value" "Conn_01x10"
-			(at 339.09 35.5599 0)
+		(property "Value" "Conn_01x09"
+			(at 339.09 34.2899 0)
 			(effects
 				(font
@@
 			)
 		)
-		(property "Description" "Generic connector, single row, 01x10, script generated (kicad-library-utils/schlib/autogen/connector/)"
+		(property "Description" "Generic connector, single row, 01x09, script generated (kicad-library-utils/schlib/autogen/connector/)"
 			(at 336.55 33.02 0)
 			(effects
@@
 		(pin "2"
 		)
-		(pin "10"
-		)
 		(instances

Commit message: Complete PCB
Parts:
- added D5: LED, LED_SMD:LED_0603_1608Metric, symbol Device:LED
- added H1, H2, H3, H4: MountingHole, MountingHole:MountingHole_3.2mm_M3, symbol Mechanical:MountingHole
- added J5, J6: Screw_Terminal_01x02, TerminalBlock:TerminalBlock_Xinya_XY308-2.54-2P_1x02_P2.54mm_Horizontal, symbol Connector:Screw_Terminal_01x02
- added R39: 10 kΩ, Resistor_SMD:R_0402_1005Metric, symbol Device:R
- added R40: 51 Ω, Resistor_SMD:R_0805_2012Metric, symbol Device:R
- added TP1, TP2, TP3: TestPoint, TestPoint:TestPoint_Pad_1.0x1.0mm, symbol Connector:TestPoint
- C1: value 4.7 µF -> 10 µF; footprint Capacitor_SMD:C_0402_1005Metric -> Capacitor_SMD:C_0805_2012Metric
- C16: value 22 µF -> 10 µF; footprint Capacitor_SMD:C_0603_1608Metric -> Capacitor_SMD:C_0805_2012Metric
- D1: Availability In Stock -> (none); Check_prices https://www.snapeda.com/parts/1N5819HW-7-F/Diodes+Inc./view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 -> (none); Description_1 Diode Schottky 1A 40V SOD123 | Diodes Inc 1N5819HW-7-F -> (none); MANUFACTURER Diodes Inc. -> (none); MF Diodes Inc. -> (none); MP 1N5819HW-7-F -> (none); PARTREV 18-2 -> (none); Package SOD-123 Fairchild Semiconductor -> (none); Price None -> (none); STANDARD IPC-7351B -> (none); SnapEDA_Link https://www.snapeda.com/parts/1N5819HW-7-F/Diodes+Inc./view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 -> (none)
- D2, D3, D4: Availability In Stock -> (none); Check_prices https://www.snapeda.com/parts/LESD5D5.0CT1G/Leshan+Radio/vi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 -> (none); Description_1 Transient Voltage Suppressors for ESD Protection -> (none); MANUFACTURER LRC -> (none); MAXIMUM_PACKAGE_HEIGHT 0.7 mm -> (none); MF Leshan Radio Co. -> (none); MP LESD5D5.0CT1G -> (none); PARTREV O -> (none); Package None -> (none); Price None -> (none); STANDARD Manufacturer Recommendations -> (none); SnapEDA_Link https://www.snapeda.com/parts/LESD5D5.0CT1G/Leshan+Radio/vi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 -> (none)
- U2: A_MAX 1.0 -> (none); Availability In Stock -> (none); B_MAX 0.45 -> (none); B_MIN 0.23 -> (none); B_NOM 0.34 -> (none); Check_prices https://www.snapeda.com/parts/LD39200PU33R/STMicroelectroni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 -> (none); D2_NOM 2.365 -> (none); D_MAX 3.1 -> (none); D_MIN 2.9 -> (none); D_NOM 3.0 -> (none); Description_1 Linear Voltage Regulator IC Positive Fixed 1 Output 2A 6-DF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 -> (none); E2_NOM 1.625 -> (none); ENOM 0.95 -> (none); E_MAX 3.1 -> (none); E_MIN 2.9 -> (none); E_NOM 3.0 -> (none); L_MAX 0.5 -> (none); L_MIN 0.3 -> (none); L_NOM 0.4 -> (none); MANUFACTURER ST Microelectronics -> (none); MAXIMUM_PACKAGE_HEIGHT 1.0mm -> (none); MF STMicroelectronics -> (none); MP LD39200PU33R -> (none); PARTREV 3 -> (none); PIN_COUNT 6.0 -> (none); Package DFN-6 STMicroelectronics -> (none); Price None -> (none); STANDARD IPC 7351B -> (none); SnapEDA_Link https://www.snapeda.com/parts/LD39200PU33R/STMicroelectroni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 -> (none)
- U3: footprint SOIC127P600X170-9N -> LMR38020FDDAR:SOIC127P600X170-9N; Height 1.7 -> (none); Manufacturer_Name Texas Instruments -> (none); Manufacturer_Part_Number LMR38020FDDAR -> (none); Mouser Part Number 595-LMR38020FDDAR -> (none); Mouser Price/Stock https://www.mouser.co.uk/ProductDetail/Texas-Instruments/LM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 -> (none)
- U4: Availability In Stock -> (none); Check_prices https://www.snapeda.com/parts/TPS2116DRLR/Texas+Instruments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 -> (none); Description_1 1.6-V to 5.5-V, 40-mΩ, 2.5-A, low-IQ, priority power multip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 -> (none); MANUFACTURER Texas Instruments -> (none); MAXIMUM_PACKAGE_HEIGHT 0.6 mm -> (none); MF Texas Instruments -> (none); MP TPS2116DRLR -> (none); PARTREV A -> (none); Package None -> (none); Price None -> (none); STANDARD IPC 7351B -> (none); SnapEDA_Link https://www.snapeda.com/parts/TPS2116DRLR/Texas+Instruments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 -> (none)
- U5: footprint SOP65P640X120-25N -> DRV8912QPWPRQ1:SOP65P640X120-25N; Height 1.2 -> (none); Manufacturer_Name Texas Instruments -> (none); Manufacturer_Part_Number DRV8912QPWPRQ1 -> (none); Mouser Part Number 595-DRV8912QPWPRQ1 -> (none); Mouser Price/Stock https://www.mouser.co.uk/ProductDetail/Texas-Instruments/DR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 -> (none)
- U6: Height 1.18 -> (none); Manufacturer_Name CEVA -> (none); Manufacturer_Part_Number BNO086 -> (none); Mouser Part Number 526-BNO086 -> (none); Mouser Price/Stock https://www.mouser.co.uk/ProductDetail/CEVA/BNO086?qs=ulEaX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 -> (none)
Connections:
- net CS is gone; now on net CS/10: U5.19 (NSCS)
- net SCL is gone; now on net SCL/9: U6.19 (H_SCL/SCK/RX)
- net SDA is gone; now on net SDA/8: U6.20 (H_SDA/H_MISO/TX)
- net +3V3: now also J6.1 (Pin_1), R40.2
- net GND: now also D5.1 (K), J5.2 (Pin_2), J6.2 (Pin_2)
- net OUT7: no longer U5.9 (OUT9)
- net OUT9: now also U5.9 (OUT9)
- net VIN: now also J5.1 (Pin_1)
- net at C4.1, C5.1, C6.1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: now also R39.1
- net at R4.2, U3.6 (PG): now also TP1.1
- net at U2.4 (PG): now also TP3.1
- net at U4.8 (ST): now also R39.2, TP2.1
- new net: D5.2 (A), R40.1
- no-connect marks 15 -> 13
