File: hardware_design/ESP32-S3_6_Motor_Driver_IMU/ESP32-S3_6_Motor_Driver_IMU.kicad_pcb (KiCad board)
At the start: 4 copper layers, 72.5 x 55 mm, 102 parts, among them J1 USB_C_Receptacle_USB2.0_16P, J2 Conn_01x09, J3 Conn_01x09, J4 Conn_01x01, J5 Screw_Terminal_01x02, J6 Screw_Terminal_01x02, SW1 3-1437565-0, SW2 3-1437565-0, U1 ESP32-S3-MINI-1, U2 LD39200PU33R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

Commit message: Make minor updates to the PCB
Parts:
- added G***: LOGO, LOGO, F.Cu at (130.5, 105.8)
Routing:
- net GND: vias 76 -> 96
